Commit message: Updated the urdf to group joints and links

File: ros2_ws/network/urdf/robot.urdf (robot description, URDF)
Before this commit: robot rectangle_with_pillars_and_rotated_cylinders_and_rectangles, 7 links, 6 joints
Links:
- removed link rectangle_left
- removed link rectangle_right
- added link bridge_left; visual box size=0.5 0.1 0.1
- added link bridge_right; visual box size=0.5 0.1 0.1
Joints:
- joint revolute_left: child rectangle_left -> bridge_left
- joint revolute_right: child rectangle_right -> bridge_right; mimic (none) -> joint=prismatic_right multiplier=1.57

Commit message: Actually got the visualization to work!

File: ros2_ws/network/urdf/robot.urdf (robot description, URDF)
Before this commit: robot rectangle_with_pillars_and_rotated_cylinders_and_rectangles, 7 links, 6 joints
Links:
- added link bridge_sum; visual box size=0.5 0.1 0.1
- added link cylinder_sum; visual cylinder length=0.2 radius=0.15
Joints:
- added joint mimic_revolute_right: type revolute, parent cylinder_right, child cylinder_sum, origin xyz=0 0 0 rpy=0 0 0, axis 0 1 0, limit lower=-1.5708 upper=1.5708 effort=10 velocity=1, mimic joint=revolute_right
- added joint revolute_sum: type revolute, parent cylinder_sum, child bridge_sum, origin xyz=0.0 0 0 rpy=0 0 0, axis 0 1 0, limit lower=-1.5708 upper=1.5708 effort=10 velocity=1, mimic joint=revolute_left multiplier=1.0

Commit message: Added images for documentation

File: ros2_ws/network/urdf/robot.urdf (robot description, URDF)
Before this commit: robot rectangle_with_pillars_and_rotated_cylinders_and_rectangles, 9 links, 8 joints
Joints:
- joint revolute_left: mimic joint=prismatic_left multiplier=-1.57 -> joint=prismatic_left multiplier=-0.77
- joint revolute_right: mimic joint=prismatic_right multiplier=1.57 -> joint=prismatic_right multiplier=0.77
- joint revolute_sum: mimic joint=revolute_left multiplier=1.0 -> joint=revolute_left
